File: 2019_01/2019_01.kicad_pcb (KiCad board)
At the start: 2 copper layers, 99.4 x 65 mm, 19 parts, among them J1 Write, J2 ISP, J3 Line, J4 Line, J5 Line, J6 Line, J7 Line, J8 Line, U1 ATmega328P-MU, Y1 Crystal

Commit message: Add logo to back side
Parts:
- added G***: LOGO, Footprints:nyampass_logo_26x7mm, B.Cu at (153.4, 91.2)
